Commit message: add riska robot

File: src/revine_description/urdf/riska.urdf.xacro (robot description, xacro)
@@ -1,4 +1,4 @@
 <?xml version="1.0"?>
-<robot name="acker"
+<robot name="riska"
   xmlns:xacro="http://ros.org/wiki/xacro">
   <xacro:arg name="is_sim" default="true" />
@@ -8,11 +8,10 @@
   <xacro:include filename="$(find revine_description)/urdf/inertial_matrix.xacro" />
   <xacro:include filename="$(find revine_description)/urdf/acker_ros2_control.xacro" />
-  <!-- Properties -->
   <xacro:property name="M_PI" value="3.1415926535897931"/>
-  <link name="base_footprint"/>
   <xacro:property name="base_link_mass" value="1.6" />
   <xacro:property name="base_link_w" value="0.30"/>
   <xacro:property name="base_link_h" value="0.15"/>
   <xacro:property name="base_link_d" value="0.10"/>
+  <link name="base_footprint"/>
   <joint name="base_joint" type="fixed">
     <parent link="base_footprint" />
@@ -21,5 +20,5 @@
   </joint>
   <link name="base_link">
-    <xacro:box_inertial m="${base_link_mass}" w="${base_link_w}" h="${base_link_h}" d="${base_link_d}" x="0" y="0" z="-0.15" />
+    <xacro:box_inertial m="${base_link_mass}" w="${base_link_w}" h="${base_link_h}" d="${base_link_d}" x=0 y=0 z="-0.15"/>
     <visual>
       <origin xyz="0 0 0" rpy="0 0 0" />
@@ -56,56 +55,9 @@
     </collision>
   </link>
-  <!-- <link name="wheel_back_left_link">
-    <visual>
-      <origin xyz="0 0 0" rpy="0 0 0" />
-      <geometry>
-        <mesh filename="package://revine_description/meshes/wheel_left_back_link.stl" />
-      </geometry>
-      <material name="black" />
-    </visual>
-    <collision>
-      <origin xyz="0 0 0" rpy="0 0 0" />
-      <geometry>
-        <mesh filename="package://revine_description/meshes/wheel_left_back_link.stl" />
-      </geometry>
-    </collision>
-  </link> -->
-  <!-- <joint name="wheel_back_left_joint" type="continuous">
-    <origin xyz="0 0 0" rpy="0 0 0" />
-    <parent link="base_link" />
-    <child link="wheel_left_back_link" />
-    <axis xyz="0 0 0" />
-  </joint> -->
-  <link name="wheel_back_left_link">
-    <!-- <inertial>
-      <origin xyz="0.213327728411634 -0.202539554308172 0.000327384188806199" rpy="0 0 0" />
-      <mass value="0.132308742016336" />
-      <inertia ixx="0.000109087078613509" ixy="8.99498920521203E-09" ixz="1.06792966043121E-08" iyy="0.000199665017441936" iyz="5.6160921837198E-09" izz="0.000109056977556842" />
-    </inertial> -->
-    <visual>
-      <origin xyz="0 0 0" rpy="0 0 3.1415926535897931" />
-      <geometry>
-        <mesh filename="package://revine_description/meshes/wheel_right_back_link.stl" />
-      </geometry>
-      <material name="black" />
-    </visual>
-    <collision>
-      <origin xyz="0 0 0" rpy="0 0 0" />
-      <geometry>
-        <mesh filename="package://revine_description/meshes/wheel_right_back_link.stl" />
-      </geometry>
-    </collision>
-  </link>
-  <joint name="wheel_back_left_joint" type="fixed">
-    <origin xyz="-0.106753653016542 0.0920004072996187 -0.0658214520621466" rpy="0 0 0" />
-    <parent link="base_link" />
-    <child link="wheel_back_left_link" />
-    <axis xyz="0 0 0" />
-  </joint>
   <joint name="base_green_joint" type="fixed">
-    <origin xyz="0 0 0" rpy="0 0 0" />
+    <origin xyz="0 0 0" rpy="0 0 0"/>
     <parent link="base_link" />
     <child link="base_green_link" />
-    <axis xyz="0 0 0" />
+    <axis xyz= "0 0 0"/>
   </joint>
 </robot>
